File: kicad/FencingAnalyzer.kicad_pcb (KiCad board)
At the start: 2 copper layers, 55.5 x 37.5 mm, 18 parts, among them IC1 PIC32MM0064GPL028-I/ML, IC2 LSM6DS33, SW1 SW_SPDT, U1 TPS61221

Commit message: Update text on silkscreen and in user interface, update for KiCad 7
Other:
- net class Default removed
- board text added: "David's Makerworks"
- board text removed: "David Rice Phoenix Falcons Fencing Club"
